File: VCO/VCO/VCO.sch (EAGLE design)
At the start: 0 parts

Commit message: Add schematic, fft, update simulation
Parts:
- added C1, C3, C5, C6, C7, C8: 100n, capacitor-wima:C5/2.5
- added C2: 10n, capacitor-wima:C5/2.5
- added C4: 100p, capacitor-wima:C2.5/2
- added D1: 1N4148DO35-10, diode:1N4148DO35-10
- added IC1, IC2: AD711N, analog-devices:AD711N
- added R1: 27K, eagle-ltspice:R0207/10
- added R2: 0R, eagle-ltspice:R0207/10
- added R3: 10K, eagle-ltspice:R0207/10
- added R4: 100K, eagle-ltspice:R0207/10
- added T1, T2: BC337, transistor:BC337
Connections:
- new net GND: C1.1, C3.1, C4.1, C5.1, C6.1, C7.2, C8.2, IC2.IN+
- new net N$1: R1.1, T1.B, T1.C, T2.B
- new net N$2: R2.2, T1.E, T2.E
- new net N$3: C2.1, D1.C, IC1.IN+, R3.2
- new net N$4: R3.1, T2.C
- new net N$5: D1.A, IC2.OUT
- new net N$7: C4.2, IC2.IN-, R4.1
- new net N$8: IC1.IN-, IC1.OUT, R4.2
- new net VCC: C2.2, C3.2, C5.2, C6.2, IC1.+VS, IC2.-VS
- new net VEE: C1.2, C7.1, C8.1, IC1.-VS, IC2.+VS, R2.1
