File: VCO/VCO/VCO.brd (EAGLE design)
At the start: 101.3 x 49.5 mm, 62 parts, among them IC1 AD711N, IC2 AD711N, IC3 AD711N, IC4 AD711N, IC5 AD711N, T1 BC337, T2 BC337

Commit message: Clean up
Parts:
- removed PAD11, PAD9: CV, wirepad:3,17/1,1
- added VCC, VEE: (no value), wirepad:3,17/1,1
- CV, GND: value CV -> (none)
- FM: value FM -> (none)
- PULSE: value PULSE -> (none)
- PW: value PW -> (none)
- PWM: value PWM -> (none)
- SAW: value SAW -> (none)
- SYNC: value SYNC -> (none)
- TUNE: value TUNE -> (none)
- moved C3 15.2 mm to (21.6, 33.0)
- moved C4 15.2 mm to (36.8, 33.0)
- moved C16 10.2 mm to (44.5, 31.8), turned to 0 degrees
- moved C17 10.2 mm to (54.6, 31.8)
- turned R18 to 180 degrees
- turned R3 to 180 degrees
- renumbered PAD1 to CV, PAD10 to GND, PAD2 to TUNE, PAD3 to FM, PAD4 to PWM, PAD5 to SYNC, PAD6 to PULSE, PAD7 to SAW, PAD8 to PW
Connections:
- net GND: now also GND.1; no longer PAD11.1
- net VCC: now also VCC.1; no longer PAD9.1
- net VEE: now also VEE.1; no longer GND.1
Routing:
- net GND: track 0.00 -> 281.0 mm
- net VCC: track 0.00 -> 227.2 mm, vias 0 -> 2
- net VEE: track 0.00 -> 188.6 mm
- net N$7: track 0.00 -> 90.9 mm
- net N$29: track 0.00 -> 66.0 mm
- net N$21: track 0.00 -> 49.6 mm
- net N$24: track 0.00 -> 41.6 mm
- net N$18: track 0.00 -> 41.1 mm
- net N$23: track 0.00 -> 38.8 mm
- net N$8: track 0.00 -> 34.3 mm
- net N$5: track 0.00 -> 33.4 mm
- net N$2: track 0.00 -> 26.0 mm
- net N$20: track 0.00 -> 25.3 mm
- net N$3: track 0.00 -> 25.0 mm
- net N$25: track 0.00 -> 21.6 mm
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- added copper zone on layer 1, net N$16
- added copper zone on layer 16, net N$19
- removed copper zone on layer 16, net GND
