File: LFO/Board/LFO.sch (EAGLE design)
At the start: 35 parts, among them IC1 AD711N, IC2 AD711N, T1 BC237, T2 BC237

Commit message: Progress LFO schematic
Parts:
- removed C6, C7: (no value), rcl:C-EU050-045X075
- removed IC2: AD711N, analog-devices:AD711N
- removed PAD2: (no value), wirepad:3,17/1,1
- added R16: (no value), pot:TRIM_EU-S75P
- added R17, R18: (no value), rcl:R-EU_0207/10
- added TRI: (no value), wirepad:3,17/1,1
- IC1: value AD711N -> TL074P; device analog-devices:AD711N -> linear:TL074P
- renumbered PAD1 to PULSE
Connections:
- new net N$19: R16.S, TRI.P
- new net N$20: R16.A, R18.2
- new net N$21: R16.E, R17.1
- net GND: now also IC1B.+IN, R18.1; no longer C6.2, C7.2, IC2.IN+
- net N$10: no longer R14.2
- net N$11: now also IC1A.+IN; no longer IC1.IN+
- net N$13: now also IC1A.OUT, R14.1; no longer IC1.OUT
- net N$16: now also IC1B.OUT, R17.2; no longer IC2.OUT, PAD2.P
- net N$17: now also IC1B.-IN, R14.2; no longer IC2.IN-, R14.1
- net N$6: now also IC1A.-IN; no longer IC1.IN-
- net VCC: now also IC1P.V+; no longer C7.1, IC1.+VS, IC2.+VS
- net VEE: now also IC1P.V-; no longer C6.1, IC1.-VS, IC2.-VS
Other:
- moved on the sheet: C5, R14, R15

Commit message: Progress LFO board
Parts:
- removed PULSE, TRI: (no value), wirepad:3,17/1,1
- added C10, C6, C7: (no value), rcl:C-EU050-045X075
- added D3, D4: 1N4004, diode:1N4004
- added R19, R20, R21, R22, R23, R24, R25, R26, R28, R29, R30, R31, R33, R34: (no value), rcl:R-EU_0207/10
- added R27, R32: (no value), pot:TRIM_EU-S75P
- added R35, R36: 10k, pot:3RP/1610N
- added T3, T4: BC237, transistor:BC237
- added X1, X2, X3, X4: 1503_02, con-lumberg:1503_02
- C3, C4: value (none) -> 100n; device rcl:C-EU050-045X075 -> capacitor-wima:C5/2.5
- R6, R7: value (none) -> 10k; device pot:TRIM_EU-S75P -> pot:3RP/1610N
Connections:
- new net N$15: R11.S, X1.2, X1.3
- new net N$18: D3.C, R23.1, T4.C
- new net N$22: C6.1, R22.2, T3.B
- new net N$23: C7.2, R20.1, T4.B
- new net N$24: C7.1, D4.A, R21.1
- new net N$25: D4.C, IC1C.-IN, R24.1, T3.C
- new net N$26: R22.1, R36.E
- new net N$27: R20.2, R36.A
- new net N$28: R35.E, R35.S, R36.S
- new net N$29: IC1C.+IN, R25.1, R26.2
- new net N$30: IC1C.OUT, R28.2, R30.1
- new net N$31: R27.A, R29.2
- new net N$32: R27.E, R28.1
- new net N$33: C10.1, IC1D.OUT, R31.1, R33.2
- new net N$34: C10.2, IC1D.-IN, R30.2, R31.2
- new net N$35: R32.A, R34.2
- new net N$36: R32.E, R33.1
- new net N$37: R27.S, X3.2, X3.3
- new net N$38: R32.S, X4.2, X4.3
- net GND: now also IC1D.+IN, R26.1, R29.1, R34.1, T3.E, T4.E, X1.1, X2.1, X3.1, X4.1; no longer C3.2, C4.2
- net N$10: now also R16.S, X2.2, X2.3; no longer PULSE.P, R11.S
- net N$19: now also C6.2, D3.A, R19.1; no longer R16.S, TRI.P
- net N$7: now also R7.E; no longer R6.E
- net N$8: now also R7.A; no longer R6.A
- net N$9: now also R6.E; no longer R7.E
- net VCC: now also R19.2, R21.2, R23.2, R24.2, R25.2; no longer C3.1, R7.A
- net VEE: no longer C4.1
Other:
- note added: "PULSE"
- note added: "TRI"
- moved on the sheet: C3, C4
