File: VCA/Board/VCA.sch (EAGLE design)
At the start: 46 parts, among them IC1 TL074P, IC2 TL074P, IC3 TL074P, IC4 TL074P, IC5 TL074P, Q1 J202, X1 1503_02, X2 1503_02, X3 1503_02

Commit message: VCA board
Parts:
- removed IC2, IC4, IC5: TL074P, linear:TL074P
- added C6, C7: 100n, capacitor-wima:C5/2.5
Connections:
- net GND: now also C6.1, C7.1
- net N$1: now also IC3B.+IN; no longer IC2A.+IN
- net N$18: now also IC3B.-IN, IC3B.OUT; no longer IC2A.-IN, IC2A.OUT
- net N$2: now also IC3C.+IN; no longer IC4A.+IN
- net N$25: now also IC3C.-IN, IC3C.OUT; no longer IC4A.-IN, IC4A.OUT
- net N$26: now also IC3D.+IN; no longer IC5A.+IN
- net N$27: now also IC3D.-IN; no longer IC5A.-IN
- net N$28: now also IC3D.OUT; no longer IC5A.OUT
- net VCC: now also C6.2
- net VEE: now also C7.2
Changed lines of the file:
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@@
 <part name="R15" library="pot" deviceset="TRIM_EU-" device="S75P"/>
 <part name="R16" library="pot" deviceset="3RP/1610N" device="" value="10k"/>
-<part name="IC2" library="linear" deviceset="TL074" device="P"/>
 <part name="IC3" library="linear" deviceset="TL074" device="P"/>
 <part name="C1" library="capacitor-wima" deviceset="C" device="5/2.5" value="100n"/>
@@
 <part name="SUPPLY21" library="supply2" deviceset="GND" device=""/>
 <part name="R19" library="pot" deviceset="TRIM_EU-" device="S75P"/>
-<part name="IC4" library="linear" deviceset="TL074" device="P"/>
-<part name="IC5" library="linear" deviceset="TL074" device="P"/>
 <part name="C5" library="capacitor-wima" deviceset="C" device="5/2.5" value="100n"/>
 <part name="R20" library="rcl" deviceset="R-EU_" device="0207/10"/>
@@
 <part name="R22" library="rcl" deviceset="R-EU_" device="0207/10"/>
 <part name="SUPPLY27" library="supply2" deviceset="GND" device=""/>
+<part name="SUPPLY22" library="supply2" deviceset="GND" device=""/>
+<part name="SUPPLY28" library="supply2" deviceset="VCC" device=""/>
+<part name="C6" library="capacitor-wima" deviceset="C" device="5/2.5" value="100n"/>
+<part name="SUPPLY29" library="supply2" deviceset="VEE" device=""/>
+<part name="SUPPLY30" library="supply2" deviceset="GND" device=""/>
+<part name="C7" library="capacitor-wima" deviceset="C" device="5/2.5" value="100n"/>
 </parts>
 <sheets>
@@
 <instance part="R15" gate="1" x="213.36" y="139.7" rot="R180"/>
 <instance part="R16" gate="G$1" x="223.52" y="116.84" rot="R90"/>
-<instance part="IC2" gate="A" x="170.18" y="154.94"/>
 <instance part="IC3" gate="A" x="223.52" y="152.4"/>
 <instance part="C1" gate="G$1" x="193.04" y="144.78" smashed="yes" rot="R180">
@@
 <instance part="SUPPLY21" gate="GND" x="236.22" y="129.54"/>
 <instance part="R19" gate="1" x="213.36" y="30.48" rot="R180"/>
-<instance part="IC4" gate="A" x="170.18" y="45.72"/>
-<instance part="IC5" gate="A" x="223.52" y="43.18"/>
 <instance part="C5" gate="G$1" x="193.04" y="35.56" smashed="yes" rot="R180">
 <attribute name="NAME" x="196.596" y="35.179" size="1.778" layer="95" rot="R180"/>
@@
 <instance part="R22" gate="G$1" x="236.22" y="38.1" rot="R270"/>
 <instance part="SUPPLY27" gate="GND" x="236.22" y="20.32"/>
+<instance part="IC3" gate="P" x="223.52" y="152.4"/>
+<instance part="SUPPLY22" gate="GND" x="228.6" y="162.56"/>
+<instance part="SUPPLY28" gate="G$1" x="223.52" y="175.26"/>
+<instance part="C6" gate="G$1" x="228.6" y="167.64" smashed="yes" rot="R180">
+<attribute name="NAME" x="232.156" y="167.259" size="1.778" layer="95" rot="R180"/>
+<attribute name="VALUE" x="234.696" y="172.339" size="1.778" layer="96" rot="R180"/>
+</instance>
+<instance part="SUPPLY29" gate="G$1" x="223.52" y="134.62" rot="R180"/>
+<instance part="SUPPLY30" gate="GND" x="228.6" y="129.54"/>
+<instance part="C7" gate="G$1" x="228.6" y="137.16" smashed="yes" rot="R180">
+<attribute name="NAME" x="232.156" y="136.779" size="1.778" layer="95" rot="R180"/>
+<attribute name="VALUE" x="234.696" y="141.859" size="1.778" layer="96" rot="R180"/>
+</instance>
+<instance part="IC3" gate="B" x="170.18" y="154.94"/>
+<instance part="IC3" gate="C" x="170.18" y="45.72"/>
+<instance part="IC3" gate="D" x="223.52" y="43.18"/>
 </instances>
 <busses>
@@
 <pinref part="SUPPLY27" gate="GND" pin="GND"/>
 </segment>
+<segment>
+<pinref part="C6" gate="G$1" pin="1"/>
+<pinref part="SUPPLY22" gate="GND" pin="GND"/>
+</segment>
+<segment>
+<pinref part="SUPPLY30" gate="GND" pin="GND"/>
+<wire x1="228.6" y1="132.08" x2="228.6" y2="134.62" width="0.1524" layer="91"/>
+<pinref part="C7" gate="G$1" pin="1"/>
+</segment>
 </net>
 <net name="VCC" class="0">
@@
 <wire x1="213.36" y1="63.5" x2="213.36" y2="60.96" width="0.1524" layer="91"/>
 </segment>
+<segment>
+<pinref part="SUPPLY28" gate="G$1" pin="VCC"/>
+<wire x1="223.52" y1="160.02" x2="223.52" y2="172.72" width="0.1524" layer="91"/>
+<wire x1="228.6" y1="172.72" x2="223.52" y2="172.72" width="0.1524" layer="91"/>
+<junction x="223.52" y="172.72"/>
+<pinref part="C6" gate="G$1" pin="2"/>
+<wire x1="223.52" y1="160.02" x2="223.52" y2="172.72" width="0.1524" layer="91"/>
+</segment>
 </net>
 <net name="VEE" class="1">
@@
 <junction x="165.1" y="96.52"/>
 <pinref part="C4" gate="G$1" pin="2"/>
+</segment>
+<segment>
+<wire x1="228.6" y1="142.24" x2="223.52" y2="142.24" width="0.1524" layer="91"/>
+<pinref part="SUPPLY29" gate="G$1" pin="VEE"/>
+<wire x1="223.52" y1="137.16" x2="223.52" y2="142.24" width="0.1524" layer="91"/>
+<wire x1="223.52" y1="142.24" x2="223.52" y2="144.78" width="0.1524" layer="91"/>
+<junction x="223.52" y="142.24"/>
+<pinref part="C7" gate="G$1" pin="2"/>
 </segment>
 </net>
@@
 <junction x="142.24" y="109.22"/>
 <wire x1="142.24" y1="109.22" x2="142.24" y2="157.48" width="0.1524" layer="91"/>
-<pinref part="IC2" gate="A" pin="+IN"/>
 <wire x1="142.24" y1="157.48" x2="162.56" y2="157.48" width="0.1524" layer="91"/>
+<pinref part="IC3" gate="B" pin="+IN"/>
 </segment>
 </net>
@@
 <junction x="132.08" y="78.74"/>
 <wire x1="132.08" y1="58.42" x2="132.08" y2="48.26" width="0.1524" layer="91"/>
-<pinref part="IC4" gate="A" pin="+IN"/>
 <wire x1="132.08" y1="48.26" x2="162.56" y2="48.26" width="0.1524" layer="91"/>
+<pinref part="IC3" gate="C" pin="+IN"/>
 </segment>
 </net>
@@
 <net name="N$18" class="0">
 <segment>
-<pinref part="IC2" gate="A" pin="-IN"/>
 <wire x1="162.56" y1="152.4" x2="160.02" y2="152.4" width="0.1524" layer="91"/>
 <wire x1="160.02" y1="152.4" x2="160.02" y2="144.78" width="0.1524" layer="91"/>
 <wire x1="160.02" y1="144.78" x2="182.88" y2="144.78" width="0.1524" layer="91"/>
 <wire x1="182.88" y1="144.78" x2="182.88" y2="154.94" width="0.1524" layer="91"/>
-<pinref part="IC2" gate="A" pin="OUT"/>
 <wire x1="182.88" y1="154.94" x2="177.8" y2="154.94" width="0.1524" layer="91"/>
 <pinref part="D2" gate="1" pin="A"/>
 <wire x1="182.88" y1="154.94" x2="185.42" y2="154.94" width="0.1524" layer="91"/>
+<pinref part="IC3" gate="B" pin="-IN"/>
+<pinref part="IC3" gate="B" pin="OUT"/>
 </segment>
 </net>
@@
 <net name="N$25" class="0">
 <segment>
-<pinref part="IC4" gate="A" pin="-IN"/>
 <wire x1="162.56" y1="43.18" x2="160.02" y2="43.18" width="0.1524" layer="91"/>
 <wire x1="160.02" y1="43.18" x2="160.02" y2="35.56" width="0.1524" layer="91"/>
 <wire x1="160.02" y1="35.56" x2="182.88" y2="35.56" width="0.1524" layer="91"/>
 <wire x1="182.88" y1="35.56" x2="182.88" y2="45.72" width="0.1524" layer="91"/>
-<pinref part="IC4" gate="A" pin="OUT"/>
 <wire x1="182.88" y1="45.72" x2="177.8" y2="45.72" width="0.1524" layer="91"/>
 <pinref part="D3" gate="1" pin="A"/>
 <wire x1="182.88" y1="45.72" x2="185.42" y2="45.72" width="0.1524" layer="91"/>
+<pinref part="IC3" gate="C" pin="-IN"/>
+<pinref part="IC3" gate="C" pin="OUT"/>
 </segment>
 </net>
 <net name="N$26" class="0">
 <segment>
-<pinref part="IC5" gate="A" pin="+IN"/>
 <wire x1="200.66" y1="45.72" x2="215.9" y2="45.72" width="0.1524" layer="91"/>
 <pinref part="R20" gate="G$1" pin="1"/>
@@
 <wire x1="190.5" y1="45.72" x2="193.04" y2="45.72" width="0.1524" layer="91"/>
 <junction x="193.04" y="45.72"/>
+<pinref part="IC3" gate="D" pin="+IN"/>
 </segment>
 </net>
@@
 <pinref part="R21" gate="G$1" pin="2"/>
 <wire x1="213.36" y1="35.56" x2="213.36" y2="40.64" width="0.1524" layer="91"/>
-<pinref part="IC5" gate="A" pin="-IN"/>
 <wire x1="213.36" y1="40.64" x2="213.36" y2="50.8" width="0.1524" layer="91"/>
 <wire x1="215.9" y1="40.64" x2="213.36" y2="40.64" width="0.1524" layer="91"/>
@@
 <wire x1="208.28" y1="30.48" x2="208.28" y2="40.64" width="0.1524" layer="91"/>
 <wire x1="208.28" y1="40.64" x2="213.36" y2="40.64" width="0.1524" layer="91"/>
+<pinref part="IC3" gate="D" pin="-IN"/>
 </segment>
 </net>
 <net name="N$28" class="0">
 <segment>
-<pinref part="IC5" gate="A" pin="OUT"/>
 <pinref part="R22" gate="G$1" pin="1"/>
 <wire x1="231.14" y1="43.18" x2="236.22" y2="43.18" width="0.1524" layer="91"/>
-</segment>
-</net>
+<pinref part="IC3" gate="D" pin="OUT"/>
+</segment>
+</net>
